Commit message: 최종 수정

File: src/my_leo_rover/my_leo_rover/maze.urdf (robot description, URDF)
Before this commit: robot maze, 129 links, 128 joints
Links:
- link wall_1: mass 0 -> None
- link wall_10: mass 0 -> None
- link wall_100: mass 0 -> None
- link wall_101: mass 0 -> None
- link wall_102: mass 0 -> None
- link wall_103: mass 0 -> None
- link wall_104: mass 0 -> None
- link wall_105: mass 0 -> None
- link wall_106: mass 0 -> None
- link wall_107: mass 0 -> None
- link wall_108: mass 0 -> None
- link wall_109: mass 0 -> None
- link wall_11: mass 0 -> None
- link wall_110: mass 0 -> None
- link wall_111: mass 0 -> None
- link wall_112: mass 0 -> None
- link wall_113: mass 0 -> None
- link wall_114: mass 0 -> None
- link wall_115: mass 0 -> None
- link wall_116: mass 0 -> None
- link wall_117: mass 0 -> None
- link wall_118: mass 0 -> None
- link wall_119: mass 0 -> None
- link wall_12: mass 0 -> None
- link wall_120: mass 0 -> None
- link wall_121: mass 0 -> None
- link wall_122: mass 0 -> None
- link wall_123: mass 0 -> None
- link wall_124: mass 0 -> None
- link wall_125: mass 0 -> None
- link wall_126: mass 0 -> None
- link wall_127: mass 0 -> None
- link wall_128: mass 0 -> None
- link wall_13: mass 0 -> None
- link wall_14: mass 0 -> None
- link wall_15: mass 0 -> None
- link wall_16: mass 0 -> None
- link wall_17: mass 0 -> None
- link wall_18: mass 0 -> None
- link wall_19: mass 0 -> None
- link wall_2: mass 0 -> None
- link wall_20: mass 0 -> None
- link wall_21: mass 0 -> None
- link wall_22: mass 0 -> None
- link wall_23: mass 0 -> None
- link wall_24: mass 0 -> None
- link wall_25: mass 0 -> None
- link wall_26: mass 0 -> None
- link wall_27: mass 0 -> None
- link wall_28: mass 0 -> None
- link wall_29: mass 0 -> None
- link wall_3: mass 0 -> None
- link wall_30: mass 0 -> None
- link wall_31: mass 0 -> None
- link wall_32: mass 0 -> None
- link wall_33: mass 0 -> None
- link wall_34: mass 0 -> None
- link wall_35: mass 0 -> None
- link wall_36: mass 0 -> None
- link wall_37: mass 0 -> None
- link wall_38: mass 0 -> None
- link wall_39: mass 0 -> None
- link wall_4: mass 0 -> None
- link wall_40: mass 0 -> None
- link wall_41: mass 0 -> None
- link wall_42: mass 0 -> None
- link wall_43: mass 0 -> None
- link wall_44: mass 0 -> None
- link wall_45: mass 0 -> None
- link wall_46: mass 0 -> None
- link wall_47: mass 0 -> None
- link wall_48: mass 0 -> None
- link wall_49: mass 0 -> None
- link wall_5: mass 0 -> None
- link wall_50: mass 0 -> None
- link wall_51: mass 0 -> None
- link wall_52: mass 0 -> None
- link wall_53: mass 0 -> None
- link wall_54: mass 0 -> None
- link wall_55: mass 0 -> None
- link wall_56: mass 0 -> None
- link wall_57: mass 0 -> None
- link wall_58: mass 0 -> None
- link wall_59: mass 0 -> None
- link wall_6: mass 0 -> None
- link wall_60: mass 0 -> None
- link wall_61: mass 0 -> None
- link wall_62: mass 0 -> None
- link wall_63: mass 0 -> None
- link wall_64: mass 0 -> None
- link wall_65: mass 0 -> None
- link wall_66: mass 0 -> None
- link wall_67: mass 0 -> None
- link wall_68: mass 0 -> None
- link wall_69: mass 0 -> None
- link wall_7: mass 0 -> None
- link wall_70: mass 0 -> None
- link wall_71: mass 0 -> None
- link wall_72: mass 0 -> None
- link wall_73: mass 0 -> None
- link wall_74: mass 0 -> None
- link wall_75: mass 0 -> None
- link wall_76: mass 0 -> None
- link wall_77: mass 0 -> None
- link wall_78: mass 0 -> None
- link wall_79: mass 0 -> None
- link wall_8: mass 0 -> None
- link wall_80: mass 0 -> None
- link wall_81: mass 0 -> None
- link wall_82: mass 0 -> None
- link wall_83: mass 0 -> None
- link wall_84: mass 0 -> None
- link wall_85: mass 0 -> None
- link wall_86: mass 0 -> None
- link wall_87: mass 0 -> None
- link wall_88: mass 0 -> None
- link wall_89: mass 0 -> None
- link wall_9: mass 0 -> None
- link wall_90: mass 0 -> None
- link wall_91: mass 0 -> None
- link wall_92: mass 0 -> None
- link wall_93: mass 0 -> None
- link wall_94: mass 0 -> None
- link wall_95: mass 0 -> None
- link wall_96: mass 0 -> None
- link wall_97: mass 0 -> None
- link wall_98: mass 0 -> None
- link wall_99: mass 0 -> None
